Commit message: added simple interface, at least 20fps

File: navisim/models/jackals/jackal_cam_depth.urdf.xacro (robot description, xacro)
@@ -231,3 +231,7 @@
     <origin xyz="0 0 1" rpy="0 0 0"/>
   </xacro:sensor_d435>
+  <xacro:include filename="$(find navisim)/models/hokuyo/hokuyo.urdf.xacro"/>
+  <xacro:sensor_hokuyo prefix="" parent="front_mount">
+    <origin xyz="0 0 0" rpy="0 0 0"/>
+  </xacro:sensor_hokuyo>
 </robot>

File: navisim/models/realsense2_description/urdf/d435_depth.macro.xacro (robot description, xacro)
@@ -146,5 +146,5 @@
           <depthImageTopicName>depth/image_raw</depthImageTopicName>
           <depthImageInfoTopicName>/depth/camera_info</depthImageInfoTopicName>
-          <pointCloudTopicName>/depth/points</pointCloudTopicName>
+          <!--pointCloudTopicName>/depth/points</pointCloudTopicName-->
           <frameName>camera_depth_optical_frame</frameName>
           <baseline>0</baseline>
