Commit message: solved depth camera issue and changed camera position

File: naviswarm_depth_v1/models/turtlebot2/sensors/r200.urdf.xacro (robot description, xacro)
@@ -14,6 +14,6 @@
   <xacro:property name="r200_bracket_length"    value="0.176" />
   <xacro:property name="r200_bracket_width"     value="0.0285" />
-  <xacro:property name="r200_cam_offset_px" value="-0.017" />
-  <xacro:property name="r200_cam_offset_py" value="0.024" />
+  <xacro:property name="r200_cam_offset_px" value="0.2" /> <!--  -0.017  -->
+  <xacro:property name="r200_cam_offset_py" value="0.024" /><!--  0.024  -->
   <xacro:property name="r200_cam_offset_pz" value="0.005" />
   <xacro:property name="r200_cam_rgb_px" value="0.005"/>
