Commit message: added crowdmove and also changed implementation

File: crowdmove/models/turtlebot2/sensors/hokuyo.urdf.xacro (robot description, xacro)
@@ -4,5 +4,5 @@
     <link name="hokuyo_link">
       <collision>
-        <origin xyz="0 0 0" rpy="0 0 0"/>
+        <origin xyz="-0.01 0 0" rpy="0 0 0"/>
         <geometry>
           <box size="0.1 0.1 0.1"/>
@@ -23,5 +23,5 @@
     <joint name="hokuyo_joint" type="fixed">
       <!--<axis xyz="0 0 1" />-->
-      <origin xyz="0.08 0 0.430" rpy="0 0 0"/>
+      <origin xyz="-0.01 0 0.430" rpy="0 0 0"/>
       <parent link="${parent}"/>
       <child link="hokuyo_link"/>
